File: Painel_UV.sch (KiCad schematic (older format))
At the start: 50 parts, among them J1 Conn_01x02_Male, J2 Screw_Terminal_01x02

Commit message: #7 e #8: Gerada a lista de materiais utilizando o plugin bom2grouped_csv
Parts:
- D1, D10, D11, D12, D13, D14, D15, D16, D17, D18, D19, D2, D20, D21, D22, D23, D24, D25, D26, D27, D28, D29, D3, D30, D31, D32, D33, D34, D35, D36, D4, D5, D6, D7, D8, D9: Description (none) -> LED UV 3,3V 40mA
- R1, R10, R11, R12, R2, R3, R4, R5, R6, R7, R8, R9: Description (none) -> 56ohms 1/8W
Changed lines of the file:
@@
 F 2 "Resistor_THT:R_Axial_DIN0207_L6.3mm_D2.5mm_P10.16mm_Horizontal" V 2730 1550 50  0001 C CNN
 F 3 "~" H 2800 1550 50  0001 C CNN
+F 4 "56ohms 1/8W" H 2800 1550 50  0001 C CNN "Description"
 	1    2800 1550
 	1    0    0    -1
@@
 F 2 "LED_THT:LED_D5.0mm" H 2800 3100 50  0001 C CNN
 F 3 "~" H 2800 3100 50  0001 C CNN
+F 4 "LED UV 3,3V 40mA" H 2800 3100 50  0001 C CNN "Description"
 	1    2800 3100
 	0    -1   -1   0
@@
 F 2 "LED_THT:LED_D5.0mm" H 2800 2600 50  0001 C CNN
 F 3 "~" H 2800 2600 50  0001 C CNN
+F 4 "LED UV 3,3V 40mA" H 2800 2600 50  0001 C CNN "Description"
 	1    2800 2600
 	0    -1   -1   0
@@
 F 2 "LED_THT:LED_D5.0mm" H 2800 2100 50  0001 C CNN
 F 3 "~" H 2800 2100 50  0001 C CNN
+F 4 "LED UV 3,3V 40mA" H 2800 2100 50  0001 C CNN "Description"
 	1    2800 2100
 	0    -1   -1   0
@@
 F 2 "Resistor_THT:R_Axial_DIN0207_L6.3mm_D2.5mm_P10.16mm_Horizontal" V 3280 1550 50  0001 C CNN
 F 3 "~" H 3350 1550 50  0001 C CNN
+F 4 "56ohms 1/8W" H 3350 1550 50  0001 C CNN "Description"
 	1    3350 1550
 	1    0    0    -1
@@
 F 2 "LED_THT:LED_D5.0mm" H 3350 3100 50  0001 C CNN
 F 3 "~" H 3350 3100 50  0001 C CNN
+F 4 "LED UV 3,3V 40mA" H 3350 3100 50  0001 C CNN "Description"
 	1    3350 3100
 	0    -1   -1   0
@@
 F 2 "LED_THT:LED_D5.0mm" H 3350 2600 50  0001 C CNN
 F 3 "~" H 3350 2600 50  0001 C CNN
+F 4 "LED UV 3,3V 40mA" H 3350 2600 50  0001 C CNN "Description"
 	1    3350 2600
 	0    -1   -1   0
@@
 F 2 "LED_THT:LED_D5.0mm" H 3350 2100 50  0001 C CNN
 F 3 "~" H 3350 2100 50  0001 C CNN
+F 4 "LED UV 3,3V 40mA" H 3350 2100 50  0001 C CNN "Description"
 	1    3350 2100
 	0    -1   -1   0
@@
 F 2 "Resistor_THT:R_Axial_DIN0207_L6.3mm_D2.5mm_P10.16mm_Horizontal" V 3830 1550 50  0001 C CNN
 F 3 "~" H 3900 1550 50  0001 C CNN
+F 4 "56ohms 1/8W" H 3900 1550 50  0001 C CNN "Description"
 	1    3900 1550
 	1    0    0    -1
@@
 F 2 "LED_THT:LED_D5.0mm" H 3900 3100 50  0001 C CNN
 F 3 "~" H 3900 3100 50  0001 C CNN
+F 4 "LED UV 3,3V 40mA" H 3900 3100 50  0001 C CNN "Description"
 	1    3900 3100
 	0    -1   -1   0
@@
 F 2 "LED_THT:LED_D5.0mm" H 3900 2600 50  0001 C CNN
 F 3 "~" H 3900 2600 50  0001 C CNN
+F 4 "LED UV 3,3V 40mA" H 3900 2600 50  0001 C CNN "Description"
 	1    3900 2600
 	0    -1   -1   0
@@
 F 2 "LED_THT:LED_D5.0mm" H 3900 2100 50  0001 C CNN
 F 3 "~" H 3900 2100 50  0001 C CNN
+F 4 "LED UV 3,3V 40mA" H 3900 2100 50  0001 C CNN "Description"
 	1    3900 2100
 	0    -1   -1   0
@@
 F 2 "Resistor_THT:R_Axial_DIN0207_L6.3mm_D2.5mm_P10.16mm_Horizontal" V 4380 1550 50  0001 C CNN
 F 3 "~" H 4450 1550 50  0001 C CNN
+F 4 "56ohms 1/8W" H 4450 1550 50  0001 C CNN "Description"
 	1    4450 1550
 	1    0    0    -1
@@
 F 2 "LED_THT:LED_D5.0mm" H 4450 3100 50  0001 C CNN
 F 3 "~" H 4450 3100 50  0001 C CNN
+F 4 "LED UV 3,3V 40mA" H 4450 3100 50  0001 C CNN "Description"
 	1    4450 3100
 	0    -1   -1   0
@@
 F 2 "LED_THT:LED_D5.0mm" H 4450 2600 50  0001 C CNN
 F 3 "~" H 4450 2600 50  0001 C CNN
+F 4 "LED UV 3,3V 40mA" H 4450 2600 50  0001 C CNN "Description"
 	1    4450 2600
 	0    -1   -1   0
@@
 F 2 "LED_THT:LED_D5.0mm" H 4450 2100 50  0001 C CNN
 F 3 "~" H 4450 2100 50  0001 C CNN
+F 4 "LED UV 3,3V 40mA" H 4450 2100 50  0001 C CNN "Description"
 	1    4450 2100
 	0    -1   -1   0
@@
 F 2 "Resistor_THT:R_Axial_DIN0207_L6.3mm_D2.5mm_P10.16mm_Horizontal" V 4930 1550 50  0001 C CNN
 F 3 "~" H 5000 1550 50  0001 C CNN
+F 4 "56ohms 1/8W" H 5000 1550 50  0001 C CNN "Description"
 	1    5000 1550
 	1    0    0    -1
@@
 F 2 "LED_THT:LED_D5.0mm" H 5000 3100 50  0001 C CNN
 F 3 "~" H 5000 3100 50  0001 C CNN
+F 4 "LED UV 3,3V 40mA" H 5000 3100 50  0001 C CNN "Description"
 	1    5000 3100
 	0    -1   -1   0
@@
 F 2 "LED_THT:LED_D5.0mm" H 5000 2600 50  0001 C CNN
 F 3 "~" H 5000 2600 50  0001 C CNN
+F 4 "LED UV 3,3V 40mA" H 5000 2600 50  0001 C CNN "Description"
 	1    5000 2600
 	0    -1   -1   0
@@
 F 2 "LED_THT:LED_D5.0mm" H 5000 2100 50  0001 C CNN
 F 3 "~" H 5000 2100 50  0001 C CNN
+F 4 "LED UV 3,3V 40mA" H 5000 2100 50  0001 C CNN "Description"
 	1    5000 2100
 	0    -1   -1   0
@@
 F 2 "Resistor_THT:R_Axial_DIN0207_L6.3mm_D2.5mm_P10.16mm_Horizontal" V 5480 1550 50  0001 C CNN
 F 3 "~" H 5550 1550 50  0001 C CNN
+F 4 "56ohms 1/8W" H 5550 1550 50  0001 C CNN "Description"
 	1    5550 1550
 	1    0    0    -1
@@
 F 2 "LED_THT:LED_D5.0mm" H 5550 3100 50  0001 C CNN
 F 3 "~" H 5550 3100 50  0001 C CNN
+F 4 "LED UV 3,3V 40mA" H 5550 3100 50  0001 C CNN "Description"
 	1    5550 3100
 	0    -1   -1   0
@@
 F 2 "LED_THT:LED_D5.0mm" H 5550 2600 50  0001 C CNN
 F 3 "~" H 5550 2600 50  0001 C CNN
+F 4 "LED UV 3,3V 40mA" H 5550 2600 50  0001 C CNN "Description"
 	1    5550 2600
 	0    -1   -1   0
@@
 F 2 "LED_THT:LED_D5.0mm" H 5550 2100 50  0001 C CNN
 F 3 "~" H 5550 2100 50  0001 C CNN
+F 4 "LED UV 3,3V 40mA" H 5550 2100 50  0001 C CNN "Description"
 	1    5550 2100
 	0    -1   -1   0
@@
 F 2 "Resistor_THT:R_Axial_DIN0207_L6.3mm_D2.5mm_P10.16mm_Horizontal" V 8780 1550 50  0001 C CNN
 F 3 "~" H 8850 1550 50  0001 C CNN
+F 4 "56ohms 1/8W" H 8850 1550 50  0001 C CNN "Description"
 	1    8850 1550
 	1    0    0    -1
@@
 F 2 "LED_THT:LED_D5.0mm" H 8850 3100 50  0001 C CNN
 F 3 "~" H 8850 3100 50  0001 C CNN
+F 4 "LED UV 3,3V 40mA" H 8850 3100 50  0001 C CNN "Description"
 	1    8850 3100
 	0    -1   -1   0
@@
 F 2 "LED_THT:LED_D5.0mm" H 8850 2600 50  0001 C CNN
 F 3 "~" H 8850 2600 50  0001 C CNN
+F 4 "LED UV 3,3V 40mA" H 8850 2600 50  0001 C CNN "Description"
 	1    8850 2600
 	0    -1   -1   0
@@
 F 2 "LED_THT:LED_D5.0mm" H 8850 2100 50  0001 C CNN
 F 3 "~" H 8850 2100 50  0001 C CNN
+F 4 "LED UV 3,3V 40mA" H 8850 2100 50  0001 C CNN "Description"
 	1    8850 2100
 	0    -1   -1   0
@@
 F 2 "Resistor_THT:R_Axial_DIN0207_L6.3mm_D2.5mm_P10.16mm_Horizontal" V 8230 1550 50  0001 C CNN
 F 3 "~" H 8300 1550 50  0001 C CNN
+F 4 "56ohms 1/8W" H 8300 1550 50  0001 C CNN "Description"
 	1    8300 1550
 	1    0    0    -1
@@
 F 2 "LED_THT:LED_D5.0mm" H 8300 3100 50  0001 C CNN
 F 3 "~" H 8300 3100 50  0001 C CNN
+F 4 "LED UV 3,3V 40mA" H 8300 3100 50  0001 C CNN "Description"
 	1    8300 3100
 	0    -1   -1   0
@@
 F 2 "LED_THT:LED_D5.0mm" H 8300 2600 50  0001 C CNN
 F 3 "~" H 8300 2600 50  0001 C CNN
+F 4 "LED UV 3,3V 40mA" H 8300 2600 50  0001 C CNN "Description"
 	1    8300 2600
 	0    -1   -1   0
@@
 F 2 "LED_THT:LED_D5.0mm" H 8300 2100 50  0001 C CNN
 F 3 "~" H 8300 2100 50  0001 C CNN
+F 4 "LED UV 3,3V 40mA" H 8300 2100 50  0001 C CNN "Description"
 	1    8300 2100
 	0    -1   -1   0
@@
 F 2 "Resistor_THT:R_Axial_DIN0207_L6.3mm_D2.5mm_P10.16mm_Horizontal" V 7680 1550 50  0001 C CNN
 F 3 "~" H 7750 1550 50  0001 C CNN
+F 4 "56ohms 1/8W" H 7750 1550 50  0001 C CNN "Description"
 	1    7750 1550
 	1    0    0    -1
@@
 F 2 "LED_THT:LED_D5.0mm" H 7750 3100 50  0001 C CNN
 F 3 "~" H 7750 3100 50  0001 C CNN
+F 4 "LED UV 3,3V 40mA" H 7750 3100 50  0001 C CNN "Description"
 	1    7750 3100
 	0    -1   -1   0
@@
 F 2 "LED_THT:LED_D5.0mm" H 7750 2600 50  0001 C CNN
 F 3 "~" H 7750 2600 50  0001 C CNN
+F 4 "LED UV 3,3V 40mA" H 7750 2600 50  0001 C CNN "Description"
 	1    7750 2600
 	0    -1   -1   0
@@
 F 2 "LED_THT:LED_D5.0mm" H 7750 2100 50  0001 C CNN
 F 3 "~" H 7750 2100 50  0001 C CNN
+F 4 "LED UV 3,3V 40mA" H 7750 2100 50  0001 C CNN "Description"
 	1    7750 2100
 	0    -1   -1   0
@@
 F 2 "Resistor_THT:R_Axial_DIN0207_L6.3mm_D2.5mm_P10.16mm_Horizontal" V 7130 1550 50  0001 C CNN
 F 3 "~" H 7200 1550 50  0001 C CNN
+F 4 "56ohms 1/8W" H 7200 1550 50  0001 C CNN "Description"
 	1    7200 1550
 	1    0    0    -1
@@
 F 2 "LED_THT:LED_D5.0mm" H 7200 3100 50  0001 C CNN
 F 3 "~" H 7200 3100 50  0001 C CNN
+F 4 "LED UV 3,3V 40mA" H 7200 3100 50  0001 C CNN "Description"
 	1    7200 3100
 	0    -1   -1   0
@@
 F 2 "LED_THT:LED_D5.0mm" H 7200 2600 50  0001 C CNN
 F 3 "~" H 7200 2600 50  0001 C CNN
+F 4 "LED UV 3,3V 40mA" H 7200 2600 50  0001 C CNN "Description"
 	1    7200 2600
 	0    -1   -1   0
@@
 F 2 "LED_THT:LED_D5.0mm" H 7200 2100 50  0001 C CNN
 F 3 "~" H 7200 2100 50  0001 C CNN
+F 4 "LED UV 3,3V 40mA" H 7200 2100 50  0001 C CNN "Description"
 	1    7200 2100
 	0    -1   -1   0
@@
 F 2 "Resistor_THT:R_Axial_DIN0207_L6.3mm_D2.5mm_P10.16mm_Horizontal" V 6580 1550 50  0001 C CNN
 F 3 "~" H 6650 1550 50  0001 C CNN
+F 4 "56ohms 1/8W" H 6650 1550 50  0001 C CNN "Description"
 	1    6650 1550
 	1    0    0    -1
@@
 F 2 "LED_THT:LED_D5.0mm" H 6650 3100 50  0001 C CNN
 F 3 "~" H 6650 3100 50  0001 C CNN
+F 4 "LED UV 3,3V 40mA" H 6650 3100 50  0001 C CNN "Description"
 	1    6650 3100
 	0    -1   -1   0
@@
 F 2 "LED_THT:LED_D5.0mm" H 6650 2600 50  0001 C CNN
 F 3 "~" H 6650 2600 50  0001 C CNN
+F 4 "LED UV 3,3V 40mA" H 6650 2600 50  0001 C CNN "Description"
 	1    6650 2600
 	0    -1   -1   0
@@
 F 2 "LED_THT:LED_D5.0mm" H 6650 2100 50  0001 C CNN
 F 3 "~" H 6650 2100 50  0001 C CNN
+F 4 "LED UV 3,3V 40mA" H 6650 2100 50  0001 C CNN "Description"
 	1    6650 2100
 	0    -1   -1   0
@@
 F 2 "Resistor_THT:R_Axial_DIN0207_L6.3mm_D2.5mm_P10.16mm_Horizontal" V 6030 1550 50  0001 C CNN
 F 3 "~" H 6100 1550 50  0001 C CNN
+F 4 "56ohms 1/8W" H 6100 1550 50  0001 C CNN "Description"
 	1    6100 1550
 	1    0    0    -1
@@
 F 2 "LED_THT:LED_D5.0mm" H 6100 3100 50  0001 C CNN
 F 3 "~" H 6100 3100 50  0001 C CNN
+F 4 "LED UV 3,3V 40mA" H 6100 3100 50  0001 C CNN "Description"
 	1    6100 3100
 	0    -1   -1   0
@@
 F 2 "LED_THT:LED_D5.0mm" H 6100 2600 50  0001 C CNN
 F 3 "~" H 6100 2600 50  0001 C CNN
+F 4 "LED UV 3,3V 40mA" H 6100 2600 50  0001 C CNN "Description"
 	1    6100 2600
 	0    -1   -1   0
@@
 F 2 "LED_THT:LED_D5.0mm" H 6100 2100 50  0001 C CNN
 F 3 "~" H 6100 2100 50  0001 C CNN
+F 4 "LED UV 3,3V 40mA" H 6100 2100 50  0001 C CNN "Description"
 	1    6100 2100
 	0    -1   -1   0
